File: minimal_adpl76030/minimal_adpl76030.kicad_pcb (KiCad board)
At the start: 4 copper layers, 15.2 x 15.2 mm, 1 part, among them U1 ADPL76030EUFD-PBF

Commit message: backup
Parts:
- added L1: 1.0 µH, inductor_footprints:74437336, F.Cu at (143.1, 86.4)
- added Q1: 60 V, transistor_footprints:TSDSON-8FL, F.Cu at (138.4, 87.8)
- added Q2: 60 V, transistor_footprints:TSDSON-8FL, F.Cu at (135.4, 92.2)
- moved U1 5.33 mm to (140.0, 93.3)
Connections:
- U1 pad 1: unconnected-(U1-TG1-Pad1) -> Net-(Q1-G)
- U1 pad 23: unconnected-(U1-SW2-Pad23) -> /SW2
- U1 pad 26: unconnected-(U1-BG1-Pad26) -> /BG1
- U1 pad 28: unconnected-(U1-SW1-Pad28) -> /SW1
- U1 pad 29: unconnected-(U1-GND-Pad29) -> GND
- U1 pad 3: unconnected-(U1-LSN-Pad3) -> Net-(U1-LSN)
- U1 pad 7: unconnected-(U1-TEST1-Pad7) -> GND
Other:
- board size 15.2 x 15.2 mm -> 15.2 x 20.3 mm

Commit message: backup
Parts:
- added Q3: 25 V, transistor_footprints:TSDSON-8FL, F.Cu at (145.9, 85.6)
- added Q4: 25 V, transistor_footprints:TSDSON-8FL, F.Cu at (145.9, 90.0)
- moved Q1 4.91 mm to (134.0, 85.6)
- moved L1 3.45 mm to (140.0, 84.9), turned to 180 degrees
- moved Q2 2.61 mm to (134.0, 90.0)
- moved U1 2.21 mm to (140.0, 91.1)
Connections:
- net Net-(Q1-G) renamed /TG1
- net Net-(U1-LSN) renamed /LSN
- Q1 pad 5: unconnected-(Q1-D-Pad5) -> /VIN
- U1 pad 2: unconnected-(U1-LSP-Pad2) -> /SW1
- U1 pad 21: unconnected-(U1-VOUT-Pad21) -> /VOUT
- U1 pad 22: unconnected-(U1-TG2-Pad22) -> /TG2
- U1 pad 25: unconnected-(U1-BG2-Pad25) -> /BG2
- U1 pad 4: unconnected-(U1-VIN-Pad4) -> /VIN
Other:
- board size 15.2 x 20.3 mm -> 20.3 x 20.3 mm

Commit message: backup
Parts:
- added C1: 1 µF, capacitor_footprints:C_0402_1005Metric, F.Cu at (145.5, 92.9)
- added C2: 100 nF, capacitor_footprints:C_0402_1005Metric, F.Cu at (138.6, 87.2)
- added C3: 100 nF, capacitor_footprints:C_0402_1005Metric, F.Cu at (141.3, 87.2)
- added C4: 2.2 nF, capacitor_footprints:C_0402_1005Metric, F.Cu at (143.3, 94.4)
- added R1: 0.005 Ω, resistor_footprints:R_2010_5025Metric, F.Cu at (136.5, 81.3)
- added R2: 0.01 Ω, resistor_footprints:R_2010_5025Metric, F.Cu at (150.6, 92.9)
- added R3: 10 kΩ, resistor_footprints:R_0402_1005Metric, F.Cu at (147.1, 92.3)
- added R4: 10 kΩ, resistor_footprints:R_0402_1005Metric, F.Cu at (147.1, 93.5)
- added R5: 10 kΩ, resistor_footprints:R_0402_1005Metric, F.Cu at (143.3, 92.3)
- moved L1 5.06 mm to (143.5, 81.3)
- moved Q1 4.13 mm to (133.2, 89.6), turned to 180 degrees
- moved Q3 4.13 mm to (146.7, 89.6), turned to 0 degrees
- moved Q2 4.13 mm to (133.2, 86.0), turned to 180 degrees
- moved Q4 4.13 mm to (146.7, 86.0), turned to 0 degrees
Connections:
- net /SW1 renamed /LSP
- U1 pad 11: unconnected-(U1-ISP-Pad11) -> /ISP
- U1 pad 12: unconnected-(U1-ISN-Pad12) -> /ISN
- U1 pad 17: unconnected-(U1-VC-Pad17) -> Net-(U1-VC)
- U1 pad 24: unconnected-(U1-BST2-Pad24) -> Net-(U1-BST2)
- U1 pad 27: unconnected-(U1-BST1-Pad27) -> Net-(U1-BST1)
Routing:
- net /LSN: track 0.00 -> 20.0 mm, vias 0 -> 2
- net /LSP: track 0.00 -> 18.3 mm, vias 0 -> 2
- net /ISP: track 0.00 -> 9.51 mm, vias 0 -> 2
- net /ISN: track 0.00 -> 8.93 mm, vias 0 -> 2
- net /BG1: track 0.00 -> 7.93 mm, vias 0 -> 2
- net /BG2: track 0.00 -> 7.54 mm, vias 0 -> 2
- net /TG2: track 0.00 -> 4.67 mm, vias 0 -> 2
- net /VOUT: track 0.00 -> 4.26 mm, vias 0 -> 3
- net /TG1: track 0.00 -> 3.83 mm, vias 0 -> 2
- net /V_OUT: track 0.00 -> 3.25 mm, vias 0 -> 2
- net Net-(U1-BST1): track 0.00 -> 1.45 mm
- net Net-(U1-BST2): track 0.00 -> 1.45 mm
- net Net-(U1-VC): track 0.00 -> 1.40 mm
- net Net-(C4-Pad1): track 0.00 -> 1.10 mm
- net /VIN: track 0.00 -> 0.94 mm, vias 0 -> 2
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- added copper zone on F.Cu, net /LSN
- added copper zone on F.Cu, net /LSP
- added copper zone on F.Cu, net /SW2
- added copper zone on In1.Cu, net /VIN
- added copper zone on F.Cu, net /VOUT
- added copper zone on F.Cu, net /V_OUT
- added copper zone on B.Cu, net GND
- added copper zone on F.Cu, net GND
- added copper zone on In2.Cu, net GND
Other:
- board size 20.3 x 20.3 mm -> 25.4 x 20.3 mm

Commit message: backup
Parts:
- added C5: 4.7 µF, capacitor_footprints:C_0603_1608Metric, F.Cu at (134.3, 92.3)
- added C6: 22 nF, capacitor_footprints:C_0402_1005Metric, F.Cu at (142.2, 95.3)
- added C7: 470 nF, capacitor_footprints:C_0402_1005Metric, F.Cu at (137.6, 94.9)
- added R10: 75 kΩ, resistor_footprints:R_0402_1005Metric, F.Cu at (138.2, 97.5)
- added R11: 110 kΩ, resistor_footprints:R_0402_1005Metric, F.Cu at (143.9, 93.3)
- added R12: 10 kΩ, resistor_footprints:R_0402_1005Metric, F.Cu at (143.9, 94.8)
- added R13: 100 kΩ, resistor_footprints:R_0402_1005Metric, F.Cu at (144.1, 90.5)
- added R6: 383 kΩ, resistor_footprints:R_0402_1005Metric, F.Cu at (134.5, 94.2)
- added R7: 165 kΩ, resistor_footprints:R_0402_1005Metric, F.Cu at (135.9, 94.2)
- added R8: 100 kΩ, resistor_footprints:R_0402_1005Metric, F.Cu at (140.5, 96.2)
- added R9: 124 kΩ, resistor_footprints:R_0402_1005Metric, F.Cu at (138.2, 96.2)
- moved C4 2.98 mm to (145.7, 92.6)
- moved C1 2.29 mm to (147.8, 92.9)
- moved R2 2.29 mm to (152.9, 92.9)
- moved R3 2.29 mm to (149.4, 92.3)
- moved R4 2.29 mm to (149.4, 93.5)
- moved Q3 1.27 mm to (148.0, 89.6)
- moved Q4 1.27 mm to (148.0, 86.0)
- moved Q1 1.27 mm to (131.9, 89.6)
- moved Q2 1.27 mm to (131.9, 86.0)
- moved R5 0.62 mm to (143.9, 92.1), turned to 0 degrees
Connections:
- net Net-(U1-BST1) renamed /BST1
- net Net-(U1-BST2) renamed /BST2
- U1 pad 10: unconnected-(U1-CTRL-Pad10) -> /CTRL
- U1 pad 14: unconnected-(U1-~{PGOOD}-Pad14) -> /~{PGOOD}
- U1 pad 15: unconnected-(U1-SS-Pad15) -> /SS
- U1 pad 16: unconnected-(U1-FB-Pad16) -> /FB
- U1 pad 18: unconnected-(U1-RT-Pad18) -> Net-(U1-RT)
- U1 pad 5: unconnected-(U1-INTVCC-Pad5) -> /INTVCC
- U1 pad 6: unconnected-(U1-EN/UVLO-Pad6) -> /EN/UVLO
- U1 pad 8: unconnected-(U1-TEST2-Pad8) -> /VREF
- U1 pad 9: unconnected-(U1-VREF-Pad9) -> /VREF
Routing:
- net /EN/UVLO: track 0.00 -> 4.52 mm
- net /VREF: track 0.00 -> 4.33 mm
- net /CTRL: track 0.00 -> 4.09 mm
- net /INTVCC: track 0.00 -> 4.07 mm, vias 0 -> 2
- net /FB: track 0.00 -> 3.41 mm
- net /~{PGOOD}: track 0.00 -> 2.80 mm
- net /ISP: track 9.51 -> 12.3 mm
- net /ISN: track 8.93 -> 11.7 mm
- net Net-(U1-RT): track 0.00 -> 2.30 mm
- net /SS: track 0.00 -> 2.20 mm
- net /VIN: track 0.94 -> 2.57 mm, vias 2 -> 3
- net /TG1: track 3.83 -> 5.10 mm
- net /BG1: track 7.93 -> 9.20 mm
- net /BG2: track 7.54 -> 8.81 mm
- net /LSN: track 20.0 -> 21.1 mm
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- added copper zone on In1.Cu, net /INTVCC
- added copper zone on In1.Cu, net /VOUT
- added copper zone on In1.Cu, net /V_OUT
Other:
- board size 25.4 x 20.3 mm -> 30.5 x 21.6 mm

Commit message: backup
Parts:
- added C10: 100 nF, capacitor_footprints:C_0402_1005Metric, F.Cu at (128.5, 88.0)
- added C11: 4.7 µF, capacitor_footprints:C_1206_3216Metric, F.Cu at (128.7, 92.0)
- added C12: 100 nF, capacitor_footprints:C_0402_1005Metric, F.Cu at (151.4, 89.3)
- added C13: 100 nF, capacitor_footprints:C_0402_1005Metric, F.Cu at (151.4, 88.0)
- added C8: 4.7 µF, capacitor_footprints:C_1206_3216Metric, F.Cu at (128.7, 94.5)
- added C9: 100 nF, capacitor_footprints:C_0402_1005Metric, F.Cu at (128.5, 89.3)
- added JP1: SolderJumper_3_Open, solder_jumper_footprints:SolderJumper-3_P1.3mm_Bridged_2_3_RoundedPad1.0x1.5mm_NumberLabels_1, F.Cu at (148.0, 97.3)
- moved C1 5.21 mm to (151.2, 96.8), turned to 0 degrees
- moved R3 3.10 mm to (150.6, 95.2), turned to -90 degrees
- moved R4 2.90 mm to (151.8, 95.2), turned to -90 degrees
- moved R10 2.59 mm to (140.4, 96.2), turned to 0 degrees
- moved R11 2.55 mm to (146.2, 94.4), turned to 90 degrees
- moved L1 1.96 mm to (141.8, 82.4), turned to 90 degrees
- moved R8 1.84 mm to (142.2, 95.7), turned to -90 degrees
- moved R2 1.83 mm to (151.2, 92.4), turned to 0 degrees
- moved C6 1.58 mm to (143.5, 94.4)
- moved R1 1.33 mm to (137.2, 82.4), turned to 90 degrees
- moved R12 1.04 mm to (144.8, 94.4), turned to 90 degrees
- moved R5 0.99 mm to (144.8, 92.3), turned to -90 degrees
- moved Q1 0.75 mm to (131.9, 88.9)
- moved Q2 0.75 mm to (131.9, 85.2)
- moved Q3 0.75 mm to (148.0, 88.9)
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Connections:
- net Net-(U1-RT) renamed /RT
- net Net-(U1-VC) renamed /VC
- U1 pad 19: unconnected-(U1-SYNC/SPRD-Pad19) -> /SYNC/SPRD
Routing:
- net /SYNC/SPRD: track 0.00 -> 9.71 mm, vias 0 -> 2
- net /ISN: track 11.7 -> 19.1 mm
- net /ISP: track 12.3 -> 19.1 mm
- net /LSN: track 21.1 -> 16.5 mm
- net /LSP: track 19.3 -> 15.4 mm
- net /VOUT: track 4.21 -> 0.92 mm, vias 4 -> 3
- net /V_OUT: track 4.01 -> 0.76 mm, vias 3 -> 2
- net /FB: track 3.41 -> 4.85 mm
- net /VC: track 1.60 -> 2.95 mm
- net /INTVCC: track 4.07 -> 5.15 mm, vias 2 -> 3
- net unconnected-(U1-SYNC/SPRD-Pad19): track 0.94 -> 0.00 mm, vias 1 -> 0
- net /BG2: track 8.81 -> 7.89 mm
- net /~{PGOOD}: track 2.80 -> 2.07 mm
- net GND: vias 3 -> 14
- added copper zone on F.Cu, net /VIN
Other:
- board size 30.5 x 21.6 mm -> 33 x 21.6 mm

Commit message: backup
Parts:
- added C14: 22 µF, capacitor_footprints:C_1206_3216Metric, F.Cu at (152.2, 84.1)
- added C15: 22 µF, capacitor_footprints:C_1206_3216Metric, F.Cu at (155.0, 84.1)
- added C16: 100 nF, capacitor_footprints:C_0402_1005Metric, F.Cu at (153.3, 96.6)
- added C17: 22 µF, capacitor_footprints:C_1206_3216Metric, F.Cu at (155.0, 96.6)
- moved C8 10.5 mm to (127.7, 84.1), turned to 90 degrees
- moved C11 8.75 mm to (124.9, 84.1), turned to 90 degrees
- moved R4 0.21 mm to (152.0, 95.2)
- moved C1 0.21 mm to (151.4, 96.8)
- moved R2 0.21 mm to (151.4, 92.4)
- moved R3 0.21 mm to (150.8, 95.2)
Routing:
- net /LSN: track 16.5 -> 15.6 mm
- net /LSP: track 15.4 -> 14.4 mm
- net /ISN: track 19.1 -> 18.4 mm
- net /ISP: track 19.1 -> 18.4 mm
- net GND: vias 14 -> 51
- net /V_OUT: vias 2 -> 10
- net /VOUT: vias 3 -> 23
- net /VIN: vias 3 -> 19
Other:
- board size 33 x 21.6 mm -> 35.6 x 22.9 mm

Commit message: backup
Parts:
- added TP1: TestPoint, test_point_footprints:TestPoint_THTPad_Castelated, F.Cu at (122.2, 82.9)
- added TP2: TestPoint, test_point_footprints:TestPoint_THTPad_Castelated, F.Cu at (122.2, 84.1)
- added TP3: TestPoint, test_point_footprints:TestPoint_THTPad_Castelated, F.Cu at (122.2, 80.3)
- added TP4: TestPoint, test_point_footprints:TestPoint_THTPad_Castelated, F.Cu at (122.2, 81.6)
- added TP5: TestPoint, test_point_footprints:TestPoint_THTPad_Castelated, F.Cu at (157.7, 84.1)
- added TP6: TestPoint, test_point_footprints:TestPoint_THTPad_Castelated, F.Cu at (157.7, 82.9)
- added TP7: TestPoint, test_point_footprints:TestPoint_THTPad_Castelated, F.Cu at (157.7, 80.3)
- added TP8: TestPoint, test_point_footprints:TestPoint_THTPad_Castelated, F.Cu at (157.7, 81.6)
- R3, R4: value 10 kΩ -> 10 Ω
- moved Q4 3.20 mm to (146.5, 82.4), turned to 90 degrees
- moved Q2 3.19 mm to (133.4, 82.4), turned to 90 degrees
- moved C8 1.91 mm to (129.6, 84.1)
- moved C14 1.91 mm to (150.3, 84.1)
- moved C15 1.91 mm to (153.1, 84.1)
- moved C11 1.90 mm to (126.8, 84.1)
- moved R1 0.35 mm to (136.9, 82.4)
Routing:
- net /BG2: track 7.77 -> 10.8 mm
- net /LSP: track 14.4 -> 13.8 mm
- net /LSN: track 15.6 -> 15.0 mm

Commit message: backup
Parts:
- added J1: CLP-104-02-G-D-BE, connector_footprints:CLP-104-02-G-D-BE, F.Cu at (162.2, 86.0)
- added J3: FW-04-03-G-D-085-155, connector_footprints:FW-04-03-G-D-085-155, F.Cu at (117.7, 82.2)
- added MB1: mouse-bite-50mil-300mil, mouse_bite_footprints:mouse-bite-50mil-300mil, F.Cu at (121.5, 82.2)
- added MB4: mouse-bite-50mil-300mil, mouse_bite_footprints:mouse-bite-50mil-300mil, F.Cu at (158.4, 86.0)
- moved TP8 6.35 mm to (157.7, 87.9)
- moved TP7 6.35 mm to (157.7, 86.7)
- moved Q1 1.93 mm to (133.4, 87.6), turned to -90 degrees
- moved Q3 1.93 mm to (146.5, 87.6), turned to -90 degrees
- moved C10 1.74 mm to (130.3, 88.4)
- moved C9 1.74 mm to (130.3, 89.7)
- moved C12 1.74 mm to (149.7, 89.7)
- moved C13 1.74 mm to (149.7, 88.4)
- moved TP5 1.27 mm to (157.7, 85.4)
- moved TP6 1.27 mm to (157.7, 84.1)
Routing:
- net /TG1: track 5.22 -> 8.56 mm
- net /TG2: track 4.96 -> 6.93 mm
- net GND: vias 51 -> 61
- net /V_OUT: vias 10 -> 20
- net /VOUT: vias 23 -> 25
- net /VIN: vias 19 -> 21
Other:
- board size 35.6 x 22.9 mm -> 52.7 x 22.9 mm
