File: minimal_adpl76030/minimal_adpl76030.kicad_pcb (KiCad board)
At the start: 4 copper layers, 52.7 x 22.9 mm, 49 parts, among them J1 CLP-104-02-G-D-BE, J3 FW-04-03-G-D-085-155, Q1 60 V, Q2 60 V, Q3 25 V, Q4 25 V, U1 ADPL76030EUFD-PBF

Commit message: backup
Parts:
- added D1: 100.0 V, diode_footprints:SOD323F, F.Cu at (136.3, 87.0)
- added D2: 100.0 V, diode_footprints:SOD323F, F.Cu at (143.7, 87.0)
- moved L1 0.72 mm to (141.8, 81.7)
- moved R1 0.72 mm to (136.9, 81.7)
- moved C2 0.40 mm to (138.1, 86.8), turned to -90 degrees
- moved C3 0.40 mm to (141.8, 86.8), turned to -90 degrees
Routing:
- net /BST2: track 1.63 -> 4.34 mm
- net /BST1: track 1.63 -> 4.34 mm
- net /INTVCC: track 5.15 -> 6.68 mm, vias 3 -> 5
- net /LSN: track 14.6 -> 15.4 mm
- net /LSP: track 13.5 -> 14.2 mm

Commit message: backup
Parts:
- moved C11 10.8 mm to (130.5, 94.2), turned to -90 degrees
- moved C8 10.3 mm to (127.7, 94.2), turned to -90 degrees
- moved J3 2.54 mm to (120.3, 82.2)
- moved TP1 2.54 mm to (124.7, 82.9)
- moved TP2 2.54 mm to (124.7, 84.1)
- moved TP3 2.54 mm to (124.7, 80.3)
- moved TP4 2.54 mm to (124.7, 81.6)
- moved MB1 2.54 mm to (124.1, 82.2)
- moved C1 0.51 mm to (151.4, 97.3)
- moved C16 0.51 mm to (153.3, 97.1)
- moved C17 0.51 mm to (155.0, 97.1)
- moved L1 0.51 mm to (141.8, 82.2)
- moved R1 0.51 mm to (136.9, 82.2)
- moved R10 0.51 mm to (140.4, 96.7)
- moved R13 0.51 mm to (143.8, 91.2)
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Other:
- board size 52.7 x 22.9 mm -> 50.2 x 22.9 mm

Commit message: backup
Parts:
- J3: value FW-04-03-G-D-085-155 -> FW-04-03-G-D-150-160; footprint connector_footprints:FW-04-03-G-D-085-155 -> connector_footprints:FW-04-03-G-D-150-160
Changed lines of the file:
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@@
 		)
 	)
-	(footprint "connector_footprints:FW-04-03-G-D-085-155"
+	(footprint "connector_footprints:FW-04-03-G-D-150-160"
 		(layer "F.Cu")
 		(at 120.269 82.21934 90)
@@
 			)
 		)
-		(property "Value" "FW-04-03-G-D-085-155"
+		(property "Value" "FW-04-03-G-D-150-160"
 			(at 0 4.572 90)
 			(unlocked yes)
@@
 			)
 		)
-		(property "Datasheet" "https://suddendocs.samtec.com/catalog_english/fw_sm.pdf?_gl=1*1xtxv9c*_gcl_au*MTM0MTYyNTQ5MS4xNzM2MDk5MTUz*_ga*MTYxNDYyMTQ0Mi4xNzM2MDk5MTUz*_ga_3KFNZC07WW*MTczODE2NTI0NS4zMi4xLjE3MzgxNjU1NjMuNjAuMC4w"
+		(property "Datasheet" "https://suddendocs.samtec.com/catalog_english/fw_sm.pdf?_gl=1*696njn*_gcl_au*OTQ3NjE2MTIwLjE3NTQ5MDMyODE.*_ga*NzIxODQzNjU3LjE3NTQ5MDMyODI.*_ga_3KFNZC07WW*czE3NTk0NzU3MTckbzkkZzEkdDE3NTk0Nzk3ODIkajYwJGwwJGgw"
 			(at 0 0 90)
 			(layer "F.Fab")
@@
 			)
 		)
-		(property "Description" "Samtec FW-xx-03-G-D-085-155 series,  4 positions connector,  1.27 mm pitch,  Black,  Vertical mounting,  5.2 A,  300 V,  Surface Mount,  Gold plated"
+		(property "Description" "Samtec FW-xx-03-G-D-150-160 series,  4 positions connector,  1.27 mm pitch,  Black,  Vertical mounting,  5.2 A,  300 V,  Surface Mount,  Gold plated"
 			(at 0 0 90)
 			(layer "F.Fab")
@@
 			)
 		)
-		(property "MPN" "FW-04-03-G-D-085-155"
+		(property "MPN" "FW-04-03-G-D-150-160"
 			(at 0 0 90)
 			(unlocked yes)
@@
 			)
 		)
-		(property "Series" "FW-xx-03-G-D-085-155"
-			(at 0 0 90)
-			(unlocked yes)
-			(layer "F.Fab")
-			(hide yes)
-			(effects
-				(font
-					(size 1 1)
-					(thickness 0.15)
-				)
-			)
-		)
-		(property "Symbol Name" "J_FW-04-03-G-D-085-155"
-			(at 0 0 90)
-			(unlocked yes)
-			(layer "F.Fab")
-			(hide yes)
-			(effects
-				(font
-					(size 1 1)
-					(thickness 0.15)
-				)
-			)
-		)
-		(property "Trustedparts Search" "https://www.trustedparts.com/en/search/FW-04-03-G-D-085-155"
+		(property "Series" "FW-xx-03-G-D-150-160"
+			(at 0 0 90)
+			(unlocked yes)
+			(layer "F.Fab")
+			(hide yes)
+			(effects
+				(font
+					(size 1 1)
+					(thickness 0.15)
+				)
+			)
+		)
+		(property "Symbol Name" "J_FW-04-03-G-D-150-160"
+			(at 0 0 90)
+			(unlocked yes)
+			(layer "F.Fab")
+			(hide yes)
+			(effects
+				(font
+					(size 1 1)
+					(thickness 0.15)
+				)
+			)
+		)
+		(property "Trustedparts Search" "https://www.trustedparts.com/en/search/FW-04-03-G-D-150-160"
 			(at 0 0 90)
 			(unlocked yes)
@@
 			(net 11 "/VIN")
 			(pintype "unspecified")
-			(teardrops
-				(best_length_ratio 0.5)
-				(max_length 1)
-				(best_width_ratio 1)
-				(max_width 2)
-				(curved_edges yes)
-				(filter_ratio 0.9)
-				(enabled yes)
-				(allow_two_segments yes)
-				(prefer_zone_connections yes)
-			)
 		)
 		(pad "2" smd roundrect
@@
 			(net 11 "/VIN")
 			(pintype "unspecified")
-			(teardrops
-				(best_length_ratio 0.5)
-				(max_length 1)
-				(best_width_ratio 1)
-				(max_width 2)
-				(curved_edges yes)
-				(filter_ratio 0.9)
-				(enabled yes)
-				(allow_two_segments yes)
-				(prefer_zone_connections yes)
-			)
 		)
 		(pad "3" smd roundrect
@@
 			(net 11 "/VIN")
 			(pintype "unspecified")
-			(teardrops
-				(best_length_ratio 0.5)
-				(max_length 1)
-				(best_width_ratio 1)
-				(max_width 2)
-				(curved_edges yes)
-				(filter_ratio 0.9)
-				(enabled yes)
-				(allow_two_segments yes)
-				(prefer_zone_connections yes)
-			)
 		)
 		(pad "4" smd roundrect
@@
 			(net 11 "/VIN")
 			(pintype "unspecified")
-			(teardrops
-				(best_length_ratio 0.5)
-				(max_length 1)
-				(best_width_ratio 1)
-				(max_width 2)
-				(curved_edges yes)
-				(filter_ratio 0.9)
-				(enabled yes)
-				(allow_two_segments yes)
-				(prefer_zone_connections yes)
-			)
 		)
 		(pad "5" smd roundrect
@@
 			(net 9 "GND")
 			(pintype "unspecified")
-			(teardrops
-				(best_length_ratio 0.5)
-				(max_length 1)
-				(best_width_ratio 1)
-				(max_width 2)
-				(curved_edges yes)
-				(filter_ratio 0.9)
-				(enabled yes)
-				(allow_two_segments yes)
-				(prefer_zone_connections yes)
-			)
 		)
 		(pad "6" smd roundrect
@@
 			(net 9 "GND")
 			(pintype "unspecified")
-			(teardrops
-				(best_length_ratio 0.5)
-				(max_length 1)
-				(best_width_ratio 1)
-				(max_width 2)
-				(curved_edges yes)
-				(filter_ratio 0.9)
-				(enabled yes)
-				(allow_two_segments yes)
-				(prefer_zone_connections yes)
-			)
 		)
 		(pad "7" smd roundrect
@@
 			(net 9 "GND")
 			(pintype "unspecified")
-			(teardrops
-				(best_length_ratio 0.5)
-				(max_length 1)
-				(best_width_ratio 1)
-				(max_width 2)
-				(curved_edges yes)
-				(filter_ratio 0.9)
-				(enabled yes)
-				(allow_two_segments yes)
-				(prefer_zone_connections yes)
-			)
 		)
 		(pad "8" smd roundrect
@@
 			(net 9 "GND")
 			(pintype "unspecified")
-			(teardrops
-				(best_length_ratio 0.5)
-				(max_length 1)
-				(best_width_ratio 1)
-				(max_width 2)
-				(curved_edges yes)
-				(filter_ratio 0.9)
-				(enabled yes)
-				(allow_two_segments yes)
-				(prefer_zone_connections yes)
-			)
 		)
 		(embedded_fonts no)
-		(model "${KICAD9_3D_MODELS_VAULT}/3D_models/connectors/FW-04-03-G-D-085-155.step"
+		(model "${KICAD9_3D_MODELS_VAULT}/3D_models/connectors/FW-04-03-G-D-150-160.step"
 			(offset
 				(xyz 0 0 0)

Commit message: backup
Parts:
- moved MB1 2.54 mm to (126.6, 82.2)
- moved J3 2.54 mm to (122.8, 82.2)
- moved TP1 2.54 mm to (127.3, 82.9)
- moved TP2 2.54 mm to (127.3, 84.1)
- moved TP3 2.54 mm to (127.3, 80.3)
- moved TP4 2.54 mm to (127.3, 81.6)
Other:
- board size 50.2 x 22.9 mm -> 47.6 x 22.9 mm

Commit message: backup
Parts:
- moved C6 7.50 mm to (156.3, 90.2), turned to 90 degrees
- moved C14 7.34 mm to (149.2, 96.2), turned to -90 degrees
- moved C15 6.12 mm to (150.8, 96.2), turned to -90 degrees
- moved C5 4.60 mm to (152.4, 89.2), turned to 0 degrees
- moved J1 2.54 mm to (125.3, 82.2)
- moved MB1 2.54 mm to (129.2, 82.2)
- moved TP1 2.54 mm to (129.8, 80.3)
- moved TP2 2.54 mm to (129.8, 81.6)
- moved TP3 2.54 mm to (129.8, 82.9)
- moved TP4 2.54 mm to (129.8, 84.1)
- moved JP1 1.37 mm to (146.8, 98.4)
- moved C1 1.27 mm to (151.6, 84.7)
- moved C11 1.27 mm to (131.8, 94.2)
- moved C13 1.27 mm to (138.9, 95.4)
- moved C17 1.27 mm to (152.6, 97.3)
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- renumbered C14 to C1, C8 to C10, C6 to C12, C7 to C13, C13 to C14, C12 to C15, C17 to C16, C1 to C17, C10 to C4, C15 to C5, C16 to C6, C9 to C7, C5 to C8, C4 to C9, J3 to J1, J1 to J2, MB4 to MB2, Q2 to Q1, Q4 to Q2, Q1 to Q3, Q3 to Q4, R4 to R10, R8 to R11, R9 to R12, R10 to R13, R13 to R2, R5 to R3, R2 to R4, R6 to R5, R7 to R6, R12 to R7, R11 to R8, R3 to R9, TP3 to TP1, TP4 to TP2, TP1 to TP3, TP2 to TP4, TP6 to TP5, TP5 to TP6
Routing:
- net /SYNC/SPRD: track 9.71 -> 8.92 mm
- net /VIN: vias 21 -> 27
- net GND: vias 61 -> 80
- net /V_OUT: vias 20 -> 21
Other:
- board size 47.6 x 22.9 mm -> 45.1 x 22.9 mm

Commit message: backup
Parts:
- R8: value 110 kΩ -> 232 kΩ
