File: minimal_adpl76030/minimal_adpl76030.kicad_sch (KiCad schematic)
At the start: 1 part, among them U1 ADPL76030EUFD-PBF

Commit message: backup
Parts:
- added L1: 1.0 µH, inductor_footprints:74437336, symbol INDUCTORS_74437336_DATA_BASE:L_74437336010
- added Q1, Q2: 60 V, transistor_footprints:TSDSON-8FL, symbol TRANSISTORS_BSZ065N06LS5ATMA1_DATA_BASE:Q_BSZ065N06LS5ATMA1
Connections:
- net at U1.1 (TG1): now also Q1.4 (G)
- net SW2: now reaches U1.23 (SW2)
- net SW2: now also L1.1
- net BG1: now reaches U1.26 (BG1)
- net BG1: now also Q2.4 (G)
- net SW1: now reaches U1.28 (SW1)
- net SW1: now also Q1.1 (S), Q1.2 (S), Q1.3 (S), Q2.1 (S), Q2.2 (S), Q2.3 (S)
- net GND: now reaches U1.29 (GND)
- net GND: now also U1.7 (TEST1), Q2.5 (D)
- net at U1.3 (LSN): now also L1.2

Commit message: backup
Parts:
- added Q3, Q4: 25 V, transistor_footprints:TSDSON-8FL, symbol TRANSISTORS_BSZ031NE2LS5ATMA1_DATA_BASE:Q_BSZ031NE2LS5ATMA1
Connections:
- net GND: now also Q4.5 (D)
- net SW1: now also U1.2 (LSP)
- net SW2: now also Q3.1 (S), Q3.2 (S), Q3.3 (S), Q4.1 (S), Q4.2 (S), Q4.3 (S)
- net TG1: now reaches Q1.4 (G), U1.1 (TG1)
- net VOUT: now reaches U1.21 (VOUT)
- net VOUT: now also Q3.5 (D)
- net TG2: now reaches U1.22 (TG2)
- net TG2: now also Q3.4 (G)
- net BG2: now reaches U1.25 (BG2)
- net BG2: now also Q4.4 (G)
- net LSN: now reaches L1.2, U1.3 (LSN)
- net VIN: now reaches U1.4 (VIN)
- net VIN: now also Q1.5 (D)
Other:
- moved on the sheet: L1, Q1, Q2

Commit message: backup
Parts:
- added C1: 1 µF, capacitor_footprints:C_0402_1005Metric, symbol CAPACITORS_C1005X6S1C_DATA_BASE:C_C1005X6S1C105K050BC
- added C2, C3: 100 nF, capacitor_footprints:C_0402_1005Metric, symbol CAPACITORS_GCM155R71H_DATA_BASE:C_GCM155R71H104KE02D
- added C4: 2.2 nF, capacitor_footprints:C_0402_1005Metric, symbol CAPACITORS_GCM155R71H_DATA_BASE:C_GCM155R71H222KA37D
- added R1: 0.005 Ω, resistor_footprints:R_2010_5025Metric, symbol RESISTORS_CRF2010-FZ-_DATA_BASE:R_CRF2010-FZ-R005ELF
- added R2: 0.01 Ω, resistor_footprints:R_2010_5025Metric, symbol RESISTORS_CRF2010-FZ-_DATA_BASE:R_CRF2010-FZ-R010ELF
- added R3, R4, R5: 10 kΩ, resistor_footprints:R_0402_1005Metric, symbol RESISTORS_ERJ-2RKF_DATA_BASE:R_ERJ-2RKF1002X
Connections:
- net GND: now also C4.2
- net LSN: now also R1.2
- net SW2: now also C3.1
- net VOUT: now also R2.1, R3.1
- net ISP: now reaches U1.11 (ISP)
- net ISP: now also C1.1, R3.2
- net ISN: now reaches U1.12 (ISN)
- net ISN: now also C1.2, R4.2
- net at U1.17 (VC): now also R5.1
- net at U1.24 (BST2): now also C3.2
- net at U1.27 (BST1): now also C2.2
- net SW1 renamed LSP
- net LSP: now also C2.1, R1.1
- new net: C4.1, R5.2
- new net V_OUT: R2.2, R4.1
Other:
- moved on the sheet: L1, Q1, Q2, Q3, Q4

Commit message: backup
Parts:
- added C5: 4.7 µF, capacitor_footprints:C_0603_1608Metric, symbol CAPACITORS_GRM188C71A_DATA_BASE:C_GRM188C71A475KE11D
- added C6: 22 nF, capacitor_footprints:C_0402_1005Metric, symbol CAPACITORS_GCM155R71H_DATA_BASE:C_GCM155R71H223KA55D
- added C7: 470 nF, capacitor_footprints:C_0402_1005Metric, symbol CAPACITORS_GCM155C71A_DATA_BASE:C_GCM155C71A474KE36D
- added R10: 75 kΩ, resistor_footprints:R_0402_1005Metric, symbol RESISTORS_ERJ-2RKF_DATA_BASE:R_ERJ-2RKF7502X
- added R11: 110 kΩ, resistor_footprints:R_0402_1005Metric, symbol RESISTORS_ERJ-2RKF_DATA_BASE:R_ERJ-2RKF1103X
- added R12: 10 kΩ, resistor_footprints:R_0402_1005Metric, symbol RESISTORS_ERJ-2RKF_DATA_BASE:R_ERJ-2RKF1002X
- added R13, R8: 100 kΩ, resistor_footprints:R_0402_1005Metric, symbol RESISTORS_ERJ-2RKF_DATA_BASE:R_ERJ-2RKF1003X
- added R6: 383 kΩ, resistor_footprints:R_0402_1005Metric, symbol RESISTORS_ERJ-2RKF_DATA_BASE:R_ERJ-2RKF3833X
- added R7: 165 kΩ, resistor_footprints:R_0402_1005Metric, symbol RESISTORS_ERJ-2RKF_DATA_BASE:R_ERJ-2RKF1653X
- added R9: 124 kΩ, resistor_footprints:R_0402_1005Metric, symbol RESISTORS_ERJ-2RKF_DATA_BASE:R_ERJ-2RKF1243X
Connections:
- net GND: now also C5.2, C6.2, C7.2, R10.2, R12.1, R13.2, R7.2
- net VIN: now also R6.1
- net V_OUT: now also R11.1
- net BST1: now reaches C2.2, U1.27 (BST1)
- net BST2: now reaches C3.2, U1.24 (BST2)
- net CTRL: now reaches U1.10 (CTRL)
- net CTRL: now also R10.1, R9.2
- net ~{PGOOD}: now reaches U1.14 (~{PGOOD})
- net ~{PGOOD}: now also R8.1
- net SS: now reaches U1.15 (SS)
- net SS: now also C6.1
- net FB: now reaches U1.16 (FB)
- net FB: now also R11.2, R12.2
- net at U1.18 (RT): now also R13.1
- net INTVCC: now reaches U1.5 (INTVCC)
- net INTVCC: now also C5.1, R8.2
- net EN/UVLO: now reaches U1.6 (EN/UVLO)
- net EN/UVLO: now also R6.2, R7.1
- net VREF: now reaches U1.8 (TEST2)
- net VREF: now also U1.9 (VREF), C7.1, R9.1
Other:
- moved on the sheet: C1, C2, C3, C4, L1, Q1, Q2, Q3, Q4, R1, R2, R3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

Commit message: backup
Parts:
- added C10, C12, C13, C9: 100 nF, capacitor_footprints:C_0402_1005Metric, symbol CAPACITORS_GCM155R71H_DATA_BASE:C_GCM155R71H104KE02D
- added C11, C8: 4.7 µF, capacitor_footprints:C_1206_3216Metric, symbol CAPACITORS_CL31B_DATA_BASE:C_CL31B475KBHNNN#
- added JP1: SolderJumper_3_Open, solder_jumper_footprints:SolderJumper-3_P1.3mm_Bridged_2_3_RoundedPad1.0x1.5mm_NumberLabels_1, symbol UNITED_SOLDER_JUMPERS:SolderJumper_3_Bridged_2_3
Connections:
- net GND: now also C10.2, C11.2, C12.2, C13.2, C8.2, C9.2, JP1.3 (B)
- net INTVCC: now also JP1.1 (A)
- net VIN: now also C10.1, C11.1, C8.1, C9.1
- net VOUT: now also C12.1, C13.1
- net RT: now reaches R13.1, U1.18 (RT)
- net VC: now reaches R5.1, U1.17 (VC)
- net SYNC/SPRD: now reaches U1.19 (SYNC/SPRD)
- net SYNC/SPRD: now also JP1.2 (C)
Other:
- moved on the sheet: C1, C2, C3, C4, C5, C6, C7, L1, Q1, Q2, Q3, Q4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

Commit message: backup
Parts:
- added C14, C15, C17: 22 µF, capacitor_footprints:C_1206_3216Metric, symbol CAPACITORS_CL31A_DATA_BASE:C_CL31A226KAHNNNE
- added C16: 100 nF, capacitor_footprints:C_0402_1005Metric, symbol CAPACITORS_GCM155R71H_DATA_BASE:C_GCM155R71H104KE02D
Connections:
- net GND: now also C14.2, C15.2, C16.2, C17.2
- net VOUT: now also C14.1, C15.1
- net V_OUT: now also C16.1, C17.1

Commit message: backup
Parts:
- added TP1, TP2, TP3, TP4, TP5, TP6, TP7, TP8: TestPoint, test_point_footprints:TestPoint_THTPad_Castelated, symbol UNITED_TEST_POINTS:TestPoint_Castelated_v2
- R3, R4: value 10 kΩ -> 10 Ω; symbol RESISTORS_ERJ-2RKF_DATA_BASE:R_ERJ-2RKF1002X -> RESISTORS_ERJ-2RKF_DATA_BASE:R_ERJ-2RKF10R0X; MPN ERJ-2RKF1002X -> ERJ-2RKF10R0X; Symbol Name R_ERJ-2RKF1002X -> R_ERJ-2RKF10R0X; Trustedparts Search https://www.trustedparts.com/en/search/ERJ-2RKF1002X -> https://www.trustedparts.com/en/search/ERJ-2RKF10R0X
Connections:
- net GND: now also TP3.1, TP4.1, TP7.1, TP8.1
- net VIN: now also TP1.1, TP2.1
- net V_OUT: now also TP5.1, TP6.1
Other:
- moved on the sheet: C3

Commit message: backup
Parts:
- added J1: CLP-104-02-G-D-BE, connector_footprints:CLP-104-02-G-D-BE, symbol CONNECTORS_CLP-1xx-02-G-D-BE_DATA_BASE:J_CLP-104-02-G-D-BE
- added J3: FW-04-03-G-D-085-155, connector_footprints:FW-04-03-G-D-085-155, symbol CONNECTORS_FW-xx-03-G-D-085-155_DATA_BASE:J_FW-04-03-G-D-085-155
- added MB1, MB4: mouse-bite-50mil-300mil, mouse_bite_footprints:mouse-bite-50mil-300mil, symbol UNITED_MOUSE_BITES_DATA_BASE:mouse-bite-50mil-300mil
Connections:
- net GND: now also J1.1, J1.2, J1.3, J1.4, J3.5, J3.6, J3.7, J3.8
- net VIN: now also J3.1, J3.2, J3.3, J3.4
- net V_OUT: now also J1.5, J1.6, J1.7, J1.8
Other:
- moved on the sheet: TP1, TP2, TP3, TP4, TP5, TP6, TP7, TP8
