File: minimal_adpl76030/minimal_adpl76030.kicad_sch (KiCad schematic)
At the start: 49 parts, among them J1 CLP-104-02-G-D-BE, J3 FW-04-03-G-D-085-155, Q1 60 V, Q2 60 V, Q3 25 V, Q4 25 V, U1 ADPL76030EUFD-PBF

Commit message: backup
Parts:
- added D1, D2: 100.0 V, diode_footprints:SOD323F, symbol DIODES_BAT46WJ,115_DATA_BASE:D_BAT46WJ,115
Connections:
- net BST1: now also D1.1
- net BST2: now also D2.1
- net INTVCC: now also D1.2, D2.2
Other:
- moved on the sheet: Q1, Q2, Q3, Q4

Commit message: backup
Parts:
- J3: value FW-04-03-G-D-085-155 -> FW-04-03-G-D-150-160; footprint connector_footprints:FW-04-03-G-D-085-155 -> connector_footprints:FW-04-03-G-D-150-160; symbol CONNECTORS_FW-xx-03-G-D-085-155_DATA_BASE:J_FW-04-03-G-D-085-155 -> CONNECTORS_FW-xx-03-G-D-150-160_DATA_BASE:J_FW-04-03-G-D-150-160; MPN FW-04-03-G-D-085-155 -> FW-04-03-G-D-150-160; Series FW-xx-03-G-D-085-155 -> FW-xx-03-G-D-150-160; Symbol Name J_FW-04-03-G-D-085-155 -> J_FW-04-03-G-D-150-160; Trustedparts Search https://www.trustedparts.com/en/search/FW-04-03-G-D-085-155 -> https://www.trustedparts.com/en/search/FW-04-03-G-D-150-160
Changed lines of the file:
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@@
 	)
 	(symbol
-		(lib_id "CONNECTORS_FW-xx-03-G-D-085-155_DATA_BASE:J_FW-04-03-G-D-085-155")
+		(lib_id "CONNECTORS_FW-xx-03-G-D-150-160_DATA_BASE:J_FW-04-03-G-D-150-160")
 		(at 88.9 120.65 0)
 		(unit 1)
@@
 			)
 		)
-		(property "Value" "FW-04-03-G-D-085-155"
+		(property "Value" "FW-04-03-G-D-150-160"
 			(at 88.9 111.76 0)
 			(effects
@@
 			)
 		)
-		(property "Footprint" "connector_footprints:FW-04-03-G-D-085-155"
+		(property "Footprint" "connector_footprints:FW-04-03-G-D-150-160"
 			(at 93.98 130.81 0)
 			(show_name yes)
@@
 			)
 		)
-		(property "Datasheet" "https://suddendocs.samtec.com/catalog_english/fw_sm.pdf?_gl=1*1xtxv9c*_gcl_au*MTM0MTYyNTQ5MS4xNzM2MDk5MTUz*_ga*MTYxNDYyMTQ0Mi4xNzM2MDk5MTUz*_ga_3KFNZC07WW*MTczODE2NTI0NS4zMi4xLjE3MzgxNjU1NjMuNjAuMC4w"
+		(property "Datasheet" "https://suddendocs.samtec.com/catalog_english/fw_sm.pdf?_gl=1*696njn*_gcl_au*OTQ3NjE2MTIwLjE3NTQ5MDMyODE.*_ga*NzIxODQzNjU3LjE3NTQ5MDMyODI.*_ga_3KFNZC07WW*czE3NTk0NzU3MTckbzkkZzEkdDE3NTk0Nzk3ODIkajYwJGwwJGgw"
 			(at 93.98 133.35 0)
 			(show_name yes)
@@
 			)
 		)
-		(property "Description" "Samtec FW-xx-03-G-D-085-155 series,  4 positions connector,  1.27 mm pitch,  Black,  Vertical mounting,  5.2 A,  300 V,  Surface Mount,  Gold plated"
+		(property "Description" "Samtec FW-xx-03-G-D-150-160 series,  4 positions connector,  1.27 mm pitch,  Black,  Vertical mounting,  5.2 A,  300 V,  Surface Mount,  Gold plated"
 			(at 93.98 135.89 0)
 			(show_name yes)
@@
 			)
 		)
-		(property "MPN" "FW-04-03-G-D-085-155"
+		(property "MPN" "FW-04-03-G-D-150-160"
 			(at 93.98 146.05 0)
 			(show_name yes)
@@
 			)
 		)
-		(property "Series" "FW-xx-03-G-D-085-155"
+		(property "Series" "FW-xx-03-G-D-150-160"
 			(at 93.98 163.83 0)
 			(show_name yes)
@@
 			)
 		)
-		(property "Symbol Name" "J_FW-04-03-G-D-085-155"
+		(property "Symbol Name" "J_FW-04-03-G-D-150-160"
 			(at 93.98 166.37 0)
 			(show_name yes)
@@
 			)
 		)
-		(property "Trustedparts Search" "https://www.trustedparts.com/en/search/FW-04-03-G-D-085-155"
+		(property "Trustedparts Search" "https://www.trustedparts.com/en/search/FW-04-03-G-D-150-160"
 			(at 93.98 168.91 0)
 			(show_name yes)

Commit message: backup
Parts:
- renumbered C14 to C1, C8 to C10, C6 to C12, C7 to C13, C13 to C14, C12 to C15, C17 to C16, C1 to C17, C10 to C4, C15 to C5, C16 to C6, C9 to C7, C5 to C8, C4 to C9, J3 to J1, J1 to J2, MB4 to MB2, Q2 to Q1, Q4 to Q2, Q1 to Q3, Q3 to Q4, R4 to R10, R8 to R11, R9 to R12, R10 to R13, R13 to R2, R5 to R3, R2 to R4, R6 to R5, R7 to R6, R12 to R7, R11 to R8, R3 to R9, TP3 to TP1, TP4 to TP2, TP1 to TP3, TP2 to TP4, TP6 to TP5, TP5 to TP6

Commit message: backup
Parts:
- R8: value 110 kΩ -> 232 kΩ; symbol RESISTORS_ERJ-2RKF_DATA_BASE:R_ERJ-2RKF1103X -> RESISTORS_ERJ-2RKF_DATA_BASE:R_ERJ-2RKF2323X; MPN ERJ-2RKF1103X -> ERJ-2RKF2323X; Symbol Name R_ERJ-2RKF1103X -> R_ERJ-2RKF2323X; Trustedparts Search https://www.trustedparts.com/en/search/ERJ-2RKF1103X -> https://www.trustedparts.com/en/search/ERJ-2RKF2323X
Changed lines of the file:
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@@
 	)
 	(symbol
-		(lib_id "RESISTORS_ERJ-2RKF_DATA_BASE:R_ERJ-2RKF1103X")
+		(lib_id "RESISTORS_ERJ-2RKF_DATA_BASE:R_ERJ-2RKF2323X")
 		(at 279.4 140.97 270)
 		(unit 1)
@@
 			)
 		)
-		(property "Value" "110 kΩ"
+		(property "Value" "232 kΩ"
 			(at 281.94 142.2399 90)
 			(effects
@@
 			)
 		)
-		(property "Description" "RES SMD 110 kΩ 1% 0402 50V"
+		(property "Description" "RES SMD 232 kΩ 1% 0402 50V"
 			(at 269.24 140.97 0)
 			(show_name yes)
@@
 			)
 		)
-		(property "MPN" "ERJ-2RKF1103X"
+		(property "MPN" "ERJ-2RKF2323X"
 			(at 259.08 140.97 0)
 			(show_name yes)
@@
 			)
 		)
-		(property "Symbol Name" "R_ERJ-2RKF1103X"
+		(property "Symbol Name" "R_ERJ-2RKF2323X"
 			(at 251.46 140.97 0)
 			(show_name yes)
@@
 			)
 		)
-		(property "Trustedparts Search" "https://www.trustedparts.com/en/search/ERJ-2RKF1103X"
+		(property "Trustedparts Search" "https://www.trustedparts.com/en/search/ERJ-2RKF2323X"
 			(at 243.84 140.97 0)
 			(show_name yes)
